Commit message: feat: urdf rover implemented, test_drive done

File: urdf/rover.urdf (robot description, URDF)
Before this commit: robot europa_explorer_v1, 5 links, 4 joints
Links:
- removed link back_left_wheel
- removed link back_right_wheel
- removed link front_left_wheel
- removed link front_right_wheel
- added link front_caster, mass 0.1; collision sphere radius=0.05; visual sphere radius=0.05
- added link left_rear_wheel, mass 0.2; collision cylinder length=0.05 radius=0.08; visual cylinder length=0.05 radius=0.08
- added link right_rear_wheel, mass 0.2; collision cylinder length=0.05 radius=0.08; visual cylinder length=0.05 radius=0.08
- link chassis: mass 50 -> 1.0; geometry collision box size=0.5 0.3 0.1; visual box size=0.5 0.3 0.1
Joints:
- removed joint back_left_wheel_joint
- removed joint back_right_wheel_joint
- removed joint front_left_wheel_joint
- removed joint front_right_wheel_joint
- added joint chassis_to_front_caster: type fixed, parent chassis, child front_caster, origin xyz=0.2 0 -0.03, axis 0 0 -1
- added joint chassis_to_left_rear_wheel: type continuous, parent chassis, child left_rear_wheel, origin xyz=-0.15 -0.175 0 rpy=1.5707 0 0, axis 0 0 -1
- added joint chassis_to_right_rear_wheel: type continuous, parent chassis, child right_rear_wheel, origin xyz=-0.15 0.175 0 rpy=1.5707 0 0, axis 0 0 -1

Commit message: feat: urdf rover dir fix

File: urdf/rover.urdf (robot description, URDF)
Before this commit: robot europa_rover, 4 links, 3 joints
Joints:
- joint chassis_to_left_rear_wheel: origin xyz=-0.15 -0.175 0 rpy=1.5707 0 0 -> xyz=-0.15 0.175 0 rpy=1.5707 0 0
- joint chassis_to_right_rear_wheel: origin xyz=-0.15 0.175 0 rpy=1.5707 0 0 -> xyz=-0.15 -0.175 0 rpy=1.5707 0 0
